File: Hardware/MCPStepper/MCPStepper.kicad_pcb (KiCad board)
At the start: 2 copper layers, 48.3 x 78 mm, 22 parts, among them J1 Conn_01x05, J2 Conn_01x05, J3 Conn_01x05, J4 Conn_01x05, J5 Conn_01x02, J6 Conn_01x05, J7 Conn_01x03, J8 Conn_01x03, J9 Conn_01x03, U1 MCP23017_SP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

Commit message: Updated the PCB
Connections:
- C2 pad 1: GND1 -> GND
- C3 pad 1: GND1 -> GND
- C4 pad 1: unconnected-(C4-Pad1) -> GND
- J5 pad 1: GND1 -> GND
- U1 pad 21: Net-(U1-Pad21) -> Net-(U3-Pad2)
- U1 pad 22: Net-(U1-Pad22) -> Net-(U3-Pad3)
- U1 pad 23: Net-(U1-Pad23) -> Net-(U3-Pad4)
- U1 pad 24: Net-(U1-Pad24) -> Net-(U3-Pad5)
- U1 pad 27: Net-(U1-Pad27) -> Net-(U4-Pad1)
- U1 pad 28: Net-(U1-Pad28) -> Net-(U4-Pad2)
- U2 pad 8: GND1 -> GND
- U3 pad 2: Net-(U1-Pad28) -> Net-(U3-Pad2)
- U3 pad 3: Net-(U1-Pad27) -> Net-(U3-Pad3)
- U3 pad 4: Net-(U1-Pad26) -> Net-(U3-Pad4)
- U3 pad 5: Net-(U1-Pad25) -> Net-(U3-Pad5)
- U3 pad 6: Net-(U1-Pad24) -> Net-(U1-Pad25)
- U3 pad 7: Net-(U1-Pad23) -> Net-(U1-Pad26)
- U3 pad 8: GND1 -> GND
- U4 pad 1: Net-(U1-Pad22) -> Net-(U4-Pad1)
- U4 pad 2: Net-(U1-Pad21) -> Net-(U4-Pad2)
- U4 pad 8: GND1 -> GND
Routing:
- net Net-(U4-Pad2): track 0.00 -> 46.0 mm
- net Net-(U4-Pad1): track 0.00 -> 40.8 mm
- net VCC: track 171.9 -> 204.9 mm
- net Net-(U1-Pad22): track 18.6 -> 0.00 mm
- net Net-(U1-Pad21): track 18.6 -> 0.00 mm
- net Net-(U3-Pad2): track 0.00 -> 18.6 mm
- net Net-(U1-Pad26): track 12.1 -> 29.4 mm
- net Net-(U3-Pad5): track 0.00 -> 16.9 mm
- net Net-(U1-Pad25): track 11.6 -> 26.5 mm
- net Net-(U3-Pad3): track 0.00 -> 14.0 mm
- net Net-(U1-Pad24): track 12.1 -> 0.00 mm
- net Net-(U1-Pad27): track 11.5 -> 0.00 mm
- net Net-(U1-Pad23): track 11.5 -> 0.00 mm
- net Net-(U1-Pad28): track 10.7 -> 0.00 mm
- net Net-(U1-Pad8): track 22.0 -> 30.0 mm
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- removed copper zone on B.Cu, net GND1
Other:
- board text added: "A0 A1 A2"
- board text added: "Gnd -- 3.3"
- board text added: "Motor Power"
- board text added: "MultiTinyStepper by Kitecraft"
- board text added: "Stepper 1"
- board text added: "Stepper 2"
- board text added: "Stepper 3"
- board text added: "Stepper 4"
- board text added: "VCC GND"
- board text added: "Vcc Gnd RST SCK SDA"

Commit message: PCB Updates
Parts:
- moved H2 92.5 mm to (166.9, 113.0), turned to 90 degrees
- moved C2 88.5 mm to (170.1, 96.0), turned to 90 degrees
- moved H5 82.6 mm to (166.9, 76.2), turned to 90 degrees
- moved J7 76.1 mm to (154.2, 111.9), turned to 90 degrees
- moved J8 74.2 mm to (154.2, 109.3), turned to 90 degrees
- moved J1 73.6 mm to (165.5, 84.1), turned to 180 degrees
- moved J9 72.5 mm to (154.2, 106.8), turned to 90 degrees
- moved J6 67.9 mm to (142.2, 117.5), turned to 90 degrees
- moved U4 62.5 mm to (149.1, 101.1), turned to 90 degrees
- moved C1 61.6 mm to (135.2, 117.6), turned to 0 degrees
- moved C3 52.2 mm to (143.8, 95.0), turned to 90 degrees
- moved J4 46.9 mm to (146.5, 84.1), turned to 180 degrees
- moved U1 45.3 mm to (117.4, 113.8), turned to 90 degrees
- moved H1 43.0 mm to (104.6, 113.0), turned to 90 degrees
- moved J5 38.2 mm to (96.5, 107.0), turned to -90 degrees
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Connections:
- J1 pad 1: VCC -> Net-(U4-Pad15)
- J1 pad 2: Net-(J1-Pad2) -> Net-(U4-Pad16)
- J1 pad 4: Net-(J1-Pad4) -> Net-(U3-Pad11)
- J1 pad 5: Net-(J1-Pad5) -> VCC
- J2 pad 1: VCC -> Net-(U2-Pad13)
- J2 pad 2: Net-(J2-Pad2) -> Net-(U2-Pad14)
- J2 pad 4: Net-(J2-Pad4) -> Net-(U2-Pad16)
- J2 pad 5: Net-(J2-Pad5) -> VCC
- J3 pad 1: VCC -> Net-(J3-Pad1)
- J3 pad 5: Net-(J3-Pad5) -> VCC
- J4 pad 1: VCC -> Net-(U3-Pad12)
- J4 pad 2: Net-(J4-Pad2) -> Net-(U3-Pad13)
- J4 pad 4: Net-(J4-Pad4) -> Net-(U3-Pad15)
- J4 pad 5: Net-(J4-Pad5) -> VCC
- U2 pad 10: Net-(J3-Pad4) -> Net-(J3-Pad2)
- U2 pad 12: Net-(J3-Pad2) -> Net-(J3-Pad4)
- U2 pad 13: Net-(J2-Pad5) -> Net-(U2-Pad13)
- U2 pad 14: Net-(J2-Pad4) -> Net-(U2-Pad14)
- U2 pad 16: Net-(J2-Pad2) -> Net-(U2-Pad16)
- U3 pad 11: Net-(J1-Pad2) -> Net-(U3-Pad11)
- U3 pad 12: Net-(J4-Pad5) -> Net-(U3-Pad12)
- U3 pad 13: Net-(J4-Pad4) -> Net-(U3-Pad13)
- U3 pad 15: Net-(J4-Pad2) -> Net-(U3-Pad15)
- U3 pad 16: Net-(J3-Pad5) -> Net-(J3-Pad1)
- U4 pad 15: Net-(J1-Pad5) -> Net-(U4-Pad15)
- U4 pad 16: Net-(J1-Pad4) -> Net-(U4-Pad16)
Routing:
- net Net-(J1-Pad2): track 29.2 -> 0.00 mm
- net Net-(U3-Pad11): track 0.00 -> 26.8 mm
- net Net-(J1-Pad4): track 21.0 -> 0.00 mm
- net Net-(J1-Pad5): track 20.3 -> 0.00 mm
- net Net-(J4-Pad5): track 19.8 -> 0.00 mm
- net Net-(J4-Pad4): track 19.7 -> 0.00 mm
- net Net-(J4-Pad2): track 19.4 -> 0.00 mm
- net Net-(U4-Pad16): track 0.00 -> 18.9 mm
- net Net-(U4-Pad15): track 0.00 -> 18.7 mm
- net Net-(U3-Pad15): track 0.00 -> 18.1 mm
- net Net-(U3-Pad13): track 0.00 -> 18.0 mm
- net Net-(U3-Pad12): track 0.00 -> 17.9 mm
- net Net-(U2-Pad16): track 0.00 -> 10.8 mm
- net Net-(J2-Pad2): track 10.8 -> 0.00 mm
- net Net-(J2-Pad4): track 10.8 -> 0.00 mm
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- added copper zone on F.Cu, net VCC
Other:
- board size 48.3 x 78 mm -> 78 x 48.3 mm
- board text added: "Address Pins"
- board text added: "Gnd"
- board text added: "Not a step"
- board text added: "This space is left intnetionally empty"
- board text added: "Vcc"
- board text added: "Vin GND"
- board text added: "|"
- board text removed: "Gnd -- 3.3"
- board text removed: "VCC GND"
