File: Hardware/MCPStepper/MCPStepper.kicad_sch (KiCad schematic)
At the start: 22 parts, among them J1 Conn_01x05, J2 Conn_01x05, J3 Conn_01x05, J4 Conn_01x05, J5 Conn_01x02, J6 Conn_01x05, J7 Conn_01x03, J8 Conn_01x03, J9 Conn_01x03, U1 MCP23017_SP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

Commit message: Updated the PCB
Connections:
- net GND1 is gone; now on net GND: C2.1, C3.1, J5.1 (Pin_1), U2.8 (GND), U3.8 (GND), U4.8 (GND)
- net GND: now also C4.1
- net at U1.21 (GPA0): now also U3.2 (I2); no longer U4.2 (I2)
- net at U1.22 (GPA1): now also U3.3 (I3); no longer U4.1 (I1)
- net at U1.23 (GPA2): now also U3.4 (I4); no longer U3.7 (I7)
- net at U1.24 (GPA3): now also U3.5 (I5); no longer U3.6 (I6)
- net at U1.25 (GPA4): now also U3.6 (I6); no longer U3.5 (I5)
- net at U1.26 (GPA5): now also U3.7 (I7); no longer U3.4 (I4)
- net at U1.27 (GPA6): now also U4.1 (I1); no longer U3.3 (I3)
- net at U1.28 (GPA7): now also U4.2 (I2); no longer U3.2 (I2)

Commit message: PCB Updates
Connections:
- net VCC: now also J1.5 (Pin_5), J2.5 (Pin_5), J3.5 (Pin_5), J4.5 (Pin_5); no longer J1.1 (Pin_1), J2.1 (Pin_1), J3.1 (Pin_1), J4.1 (Pin_1)
- net at U2.10 (O7): now also J3.2 (Pin_2); no longer J3.4 (Pin_4)
- net at U2.12 (O5): now also J3.4 (Pin_4); no longer J3.2 (Pin_2)
- net at U2.13 (O4): now also J2.1 (Pin_1); no longer J2.5 (Pin_5)
- net at U2.14 (O3): now also J2.2 (Pin_2); no longer J2.4 (Pin_4)
- net at U2.16 (O1): now also J2.4 (Pin_4); no longer J2.2 (Pin_2)
- net at U3.11 (O6): now also J1.4 (Pin_4); no longer J1.2 (Pin_2)
- net at U3.12 (O5): now also J4.1 (Pin_1); no longer J4.5 (Pin_5)
- net at U3.13 (O4): now also J4.2 (Pin_2); no longer J4.4 (Pin_4)
- net at U3.15 (O2): now also J4.4 (Pin_4); no longer J4.2 (Pin_2)
- net at U3.16 (O1): now also J3.1 (Pin_1); no longer J3.5 (Pin_5)
- net at U4.15 (O2): now also J1.1 (Pin_1); no longer J1.5 (Pin_5)
- net at U4.16 (O1): now also J1.2 (Pin_2); no longer J1.4 (Pin_4)
Changed lines of the file:
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@@
   (symbol (lib_id "power:GND") (at 163.83 16.51 90) (unit 1)
     (in_bom yes) (on_board yes)
-    (property "Reference" "#PWR?" (id 0) (at 170.18 16.51 0)
+    (property "Reference" "#PWR0112" (id 0) (at 170.18 16.51 0)
       (effects (font (size 1.27 1.27)) hide)
     )
@@
     (pin "3")
   )
-  (symbol (lib_id "Connector_Generic:Conn_01x05") (at 176.53 33.02 0) (unit 1)
-    (in_bom yes) (on_board yes) (fields_autoplaced)
-    (property "Reference" "J2" (id 0) (at 178.562 32.1853 0)
-      (effects (font (size 1.27 1.27)) (justify left))
-    )
-    (property "Value" "Conn_01x05" (id 1) (at 178.562 34.7222 0)
-      (effects (font (size 1.27 1.27)) (justify left))
-    )
+  (symbol (lib_id "Connector_Generic:Conn_01x05") (at 176.53 33.02 0) (mirror x) (unit 1)
+    (in_bom yes) (on_board yes) (fields_autoplaced)
+    (property "Reference" "J2" (id 0) (at 176.53 22.9702 0))
+    (property "Value" "Conn_01x05" (id 1) (at 176.53 25.5071 0))
     (property "Footprint" "Connector_JST:JST_XH_B5B-XH-A_1x05_P2.50mm_Vertical" (id 2) (at 176.53 33.02 0)
       (effects (font (size 1.27 1.27)) hide)
@@
     (pin "9")
   )
-  (symbol (lib_id "Connector_Generic:Conn_01x05") (at 222.25 124.46 0) (unit 1)
-    (in_bom yes) (on_board yes) (fields_autoplaced)
-    (property "Reference" "J1" (id 0) (at 224.282 123.6253 0)
-      (effects (font (size 1.27 1.27)) (justify left))
-    )
-    (property "Value" "Conn_01x05" (id 1) (at 224.282 126.1622 0)
-      (effects (font (size 1.27 1.27)) (justify left))
-    )
+  (symbol (lib_id "Connector_Generic:Conn_01x05") (at 222.25 124.46 0) (mirror x) (unit 1)
+    (in_bom yes) (on_board yes) (fields_autoplaced)
+    (property "Reference" "J1" (id 0) (at 222.25 114.4102 0))
+    (property "Value" "Conn_01x05" (id 1) (at 222.25 116.9471 0))
     (property "Footprint" "Connector_JST:JST_XH_B5B-XH-A_1x05_P2.50mm_Vertical" (id 2) (at 222.25 124.46 0)
       (effects (font (size 1.27 1.27)) hide)
@@
     (pin "1")
   )
-  (symbol (lib_id "Connector_Generic:Conn_01x05") (at 199.39 52.07 0) (unit 1)
-    (in_bom yes) (on_board yes) (fields_autoplaced)
-    (property "Reference" "J3" (id 0) (at 201.422 51.2353 0)
-      (effects (font (size 1.27 1.27)) (justify left))
-    )
-    (property "Value" "Conn_01x05" (id 1) (at 201.422 53.7722 0)
+  (symbol (lib_id "Connector_Generic:Conn_01x05") (at 199.39 52.07 0) (mirror x) (unit 1)
+    (in_bom yes) (on_board yes) (fields_autoplaced)
+    (property "Reference" "J3" (id 0) (at 201.422 52.9047 0)
+      (effects (font (size 1.27 1.27)) (justify left))
+    )
+    (property "Value" "Conn_01x05" (id 1) (at 201.422 50.3678 0)
       (effects (font (size 1.27 1.27)) (justify left))
     )
@@
   (symbol (lib_id "power:GND") (at 165.1 78.74 90) (unit 1)
     (in_bom yes) (on_board yes)
-    (property "Reference" "#PWR?" (id 0) (at 171.45 78.74 0)
+    (property "Reference" "#PWR0110" (id 0) (at 171.45 78.74 0)
       (effects (font (size 1.27 1.27)) hide)
     )
@@
     (pin "1")
   )
-  (symbol (lib_id "Connector_Generic:Conn_01x05") (at 219.71 97.79 0) (unit 1)
-    (in_bom yes) (on_board yes) (fields_autoplaced)
-    (property "Reference" "J4" (id 0) (at 221.742 96.9553 0)
-      (effects (font (size 1.27 1.27)) (justify left))
-    )
-    (property "Value" "Conn_01x05" (id 1) (at 221.742 99.4922 0)
-      (effects (font (size 1.27 1.27)) (justify left))
-    )
+  (symbol (lib_id "Connector_Generic:Conn_01x05") (at 219.71 97.79 0) (mirror x) (unit 1)
+    (in_bom yes) (on_board yes) (fields_autoplaced)
+    (property "Reference" "J4" (id 0) (at 219.71 87.7402 0))
+    (property "Value" "Conn_01x05" (id 1) (at 219.71 90.2771 0))
     (property "Footprint" "Connector_JST:JST_XH_B5B-XH-A_1x05_P2.50mm_Vertical" (id 2) (at 219.71 97.79 0)
       (effects (font (size 1.27 1.27)) hide)
@@
   (symbol (lib_id "power:GND") (at 165.1 125.73 90) (unit 1)
     (in_bom yes) (on_board yes)
-    (property "Reference" "#PWR?" (id 0) (at 171.45 125.73 0)
+    (property "Reference" "#PWR0107" (id 0) (at 171.45 125.73 0)
       (effects (font (size 1.27 1.27)) hide)
     )
@@
       (reference "#PWR0106") (unit 1) (value "GND") (footprint "")
     )
+    (path "/f1e01d27-aaa8-4b75-9b2a-0ed359bd8841"
+      (reference "#PWR0107") (unit 1) (value "GND") (footprint "")
+    )
     (path "/7bfc4649-7720-4e04-9a81-baf4232ce0d8"
       (reference "#PWR0108") (unit 1) (value "VCC") (footprint "")
@@
       (reference "#PWR0109") (unit 1) (value "VCC") (footprint "")
     )
+    (path "/d50a84f4-9a62-423e-a8cd-b3898c1fb174"
+      (reference "#PWR0110") (unit 1) (value "GND") (footprint "")
+    )
     (path "/8082776c-c914-47d0-9e37-74a918928e2c"
       (reference "#PWR0111") (unit 1) (value "GND") (footprint "")
     )
+    (path "/0d2ebbcf-e664-4983-b2b0-f971628c31bd"
+      (reference "#PWR0112") (unit 1) (value "GND") (footprint "")
+    )
     (path "/f138011e-dec6-492b-9a02-7836728d0b45"
       (reference "#PWR0113") (unit 1) (value "VCC") (footprint "")
@@
       (reference "#PWR0126") (unit 1) (value "VCC") (footprint "")
     )
-    (path "/0d2ebbcf-e664-4983-b2b0-f971628c31bd"
-      (reference "#PWR?") (unit 1) (value "GND") (footprint "")
-    )
-    (path "/d50a84f4-9a62-423e-a8cd-b3898c1fb174"
-      (reference "#PWR?") (unit 1) (value "GND") (footprint "")
-    )
-    (path "/f1e01d27-aaa8-4b75-9b2a-0ed359bd8841"
-      (reference "#PWR?") (unit 1) (value "GND") (footprint "")
-    )
     (path "/de466835-9682-4161-bd7d-a6a1ec3c7ef9"
